Commit message: modify xacro to add load_gripper argument

File: robots/panda.gazebo.xacro (robot description, xacro)
@@ -1,5 +1,5 @@
 <?xml version="1.0"?>
 <robot xmlns:xacro="http://www.ros.org/wiki/xacro">
-    <xacro:macro name="panda_gazebo" params="robot_name">
+    <xacro:macro name="panda_gazebo" params="robot_name load_gripper">
         <!-- Link0 -->
         <gazebo reference="${robot_name}_link0">
@@ -62,16 +62,18 @@
             <mu2>0.2</mu2>
         </gazebo>
-        <!-- LinkRightFinger -->
-        <gazebo reference="${robot_name}_rightfinger">
-            <material>Gazebo/Grey</material>
-            <mu1>0.2</mu1>
-            <mu2>0.2</mu2>
-        </gazebo>
-        <!-- LinkLeftFinger -->
-        <gazebo reference="${robot_name}_leftfinger">
-            <material>Gazebo/Grey</material>
-            <mu1>0.2</mu1>
-            <mu2>0.2</mu2>
-        </gazebo>
+        <xacro:if value="${load_gripper}">
+            <!-- LinkRightFinger -->
+            <gazebo reference="${robot_name}_rightfinger">
+                <material>Gazebo/Grey</material>
+                <mu1>0.2</mu1>
+                <mu2>0.2</mu2>
+            </gazebo>
+            <!-- LinkLeftFinger -->
+            <gazebo reference="${robot_name}_leftfinger">
+                <material>Gazebo/Grey</material>
+                <mu1>0.2</mu1>
+                <mu2>0.2</mu2>
+            </gazebo>
+        </xacro:if>
       <gazebo reference="${robot_name}_joint7">
         <implicitSpringDamper>1</implicitSpringDamper>
@@ -102,12 +104,14 @@
         <provideFeedback>true</provideFeedback>
       </gazebo>
-      <gazebo reference="${robot_name}_finger_joint1">
-        <implicitSpringDamper>1</implicitSpringDamper>
-        <provideFeedback>true</provideFeedback>
-      </gazebo>
-      <gazebo reference="${robot_name}_finger_joint2">
-        <implicitSpringDamper>1</implicitSpringDamper>
-        <provideFeedback>true</provideFeedback>
-      </gazebo>
+      <xacro:if value="${load_gripper}">
+          <gazebo reference="${robot_name}_finger_joint1">
+            <implicitSpringDamper>1</implicitSpringDamper>
+            <provideFeedback>true</provideFeedback>
+          </gazebo>
+          <gazebo reference="${robot_name}_finger_joint2">
+            <implicitSpringDamper>1</implicitSpringDamper>
+            <provideFeedback>true</provideFeedback>
+          </gazebo>
+      </xacro:if>
     </xacro:macro>
 </robot>

File: robots/panda.transmission.xacro (robot description, xacro)
@@ -1,5 +1,5 @@
 <?xml version="1.0"?>
 <robot xmlns:xacro="http://www.ros.org/wiki/xacro">
-    <xacro:macro name="panda_transmission" params="robot_name">
+    <xacro:macro name="panda_transmission" params="robot_name load_gripper">
         <!-- Load Gazebo lib and set the robot namespace -->
         <gazebo>
@@ -86,24 +86,26 @@
             </actuator>
         </transmission>
-        <transmission name="${robot_name}_leftfinger">
-            <type>transmission_interface/SimpleTransmission</type>
-            <joint name="${robot_name}_finger_joint1">
-                <hardwareInterface>hardware_interface/EffortJointInterface</hardwareInterface>
-            </joint>
-            <actuator name="${robot_name}_finger_joint1">
-                <hardwareInterface>hardware_interface/EffortJointInterface</hardwareInterface>
-                <mechanicalReduction>1</mechanicalReduction>
-            </actuator>
-        </transmission>
-        <transmission name="${robot_name}_rightfinger">
-            <type>transmission_interface/SimpleTransmission</type>
-            <joint name="${robot_name}_finger_joint2">
-                <hardwareInterface>hardware_interface/EffortJointInterface</hardwareInterface>
-            </joint>
-            <actuator name="${robot_name}_finger_joint2">
-                <hardwareInterface>hardware_interface/EffortJointInterface</hardwareInterface>
-                <mechanicalReduction>1</mechanicalReduction>
-            </actuator>
-        </transmission>
+        <xacro:if value="${load_gripper}">
+            <transmission name="${robot_name}_leftfinger">
+                <type>transmission_interface/SimpleTransmission</type>
+                <joint name="${robot_name}_finger_joint1">
+                    <hardwareInterface>hardware_interface/EffortJointInterface</hardwareInterface>
+                </joint>
+                <actuator name="${robot_name}_finger_joint1">
+                    <hardwareInterface>hardware_interface/EffortJointInterface</hardwareInterface>
+                    <mechanicalReduction>1</mechanicalReduction>
+                </actuator>
+            </transmission>
+            <transmission name="${robot_name}_rightfinger">
+                <type>transmission_interface/SimpleTransmission</type>
+                <joint name="${robot_name}_finger_joint2">
+                    <hardwareInterface>hardware_interface/EffortJointInterface</hardwareInterface>
+                </joint>
+                <actuator name="${robot_name}_finger_joint2">
+                    <hardwareInterface>hardware_interface/EffortJointInterface</hardwareInterface>
+                    <mechanicalReduction>1</mechanicalReduction>
+                </actuator>
+            </transmission>
+        </xacro:if>
     </xacro:macro>
 </robot>

File: robots/panda_arm_hand.urdf.xacro (robot description, xacro)
@@ -2,11 +2,14 @@
 <robot xmlns:xacro="http://www.ros.org/wiki/xacro" name="panda">
   <xacro:arg name="robot_name" default="panda"/>
+  <xacro:arg name="load_gripper" default="true"/>
   <xacro:include filename="$(find franka_panda_description)/robots/panda_arm.xacro"/>
-  <xacro:include filename="$(find franka_panda_description)/robots/hand.xacro"/>
+  <xacro:if value="$(arg load_gripper)">
+    <xacro:include filename="$(find franka_panda_description)/robots/hand.xacro"/>
+    <xacro:hand ns="panda" rpy="0 0 ${-pi/4}" connected_to="panda_link8"/>
+  </xacro:if>
   <xacro:include filename="$(find franka_panda_description)/robots/panda.gazebo.xacro"/>
   <xacro:include filename="$(find franka_panda_description)/robots/panda.transmission.xacro"/>
   <xacro:panda_arm />
-  <xacro:hand ns="panda" rpy="0 0 ${-pi/4}" connected_to="panda_link8"/>
-  <xacro:panda_gazebo robot_name="$(arg robot_name)" />
-  <xacro:panda_transmission robot_name="$(arg robot_name)" />
+  <xacro:panda_gazebo robot_name="$(arg robot_name)" load_gripper="$(arg load_gripper)"/>
+  <xacro:panda_transmission robot_name="$(arg robot_name)" load_gripper="$(arg load_gripper)"/>
 </robot>

Commit message: updates to robot description outside gazebo for KDL; adding better dynamic values for links enabling inertia matrix estimation

File: robots/panda.gazebo.xacro (robot description, xacro)
@@ -2,5 +2,4 @@
 <robot xmlns:xacro="http://www.ros.org/wiki/xacro">
     <xacro:macro name="panda_gazebo" params="robot_name load_gripper">
-        <!-- Link0 -->
         <gazebo reference="${robot_name}_link0">
             <material>Gazebo/Grey</material>

File: robots/panda_arm.urdf.xacro (robot description, xacro)
@@ -1,5 +1,11 @@
 <?xml version='1.0' ?>
 <robot xmlns:xacro="http://www.ros.org/wiki/xacro" name="panda">
-  <xacro:include filename="$(find franka_panda_description)/robots/panda_arm.xacro" />
-  <xacro:panda_arm />
+    <xacro:arg name="load_gazebo" default="false"/>
+    <xacro:include filename="$(find franka_panda_description)/robots/panda_arm.xacro"/>
+    <xacro:if value="$(arg load_gazebo)">
+        <xacro:panda_arm in_gazebo="true" />
+    </xacro:if>
+    <xacro:unless value="$(arg load_gazebo)">
+        <xacro:panda_arm />
+    </xacro:unless>
 </robot>

File: robots/panda_arm.xacro (robot description, xacro)
@@ -1,5 +1,5 @@
 <?xml version='1.0'?>
 <robot xmlns:xacro="http://www.ros.org/wiki/xacro" name="panda">
-  <xacro:macro name="panda_arm" params="arm_id:='panda' description_pkg:='franka_panda_description' connected_to:='' xyz:='0 0 0' rpy:='0 0 0'">
+  <xacro:macro name="panda_arm" params="arm_id:='panda' description_pkg:='franka_description' connected_to:=''  in_gazebo='false' xyz:='0 0 0' rpy:='0 0 0'">
     <xacro:unless value="${not connected_to}">
       <joint name="${arm_id}_joint_${connected_to}" type="fixed">
@@ -10,11 +10,13 @@
     </xacro:unless>
     <xacro:property name="joint_damping" value="1.0"/>
-    <link name="world" />
-    <joint name="robot_to_world" type="fixed">
-      <parent link="world" />
-      <child link="${arm_id}_link0" />
-      <origin xyz="0.0 0.0 0.0" rpy="0.0 0.0 0.0" />
-      <dynamics damping="${joint_damping}"/>
-    </joint>
+    <xacro:unless value="${in_gazebo == 'false'}">
+      <link name="world" />
+      <joint name="robot_to_world" type="fixed">
+        <parent link="world" />
+        <child link="${arm_id}_link0" />
+        <origin xyz="0.0 0.0 0.0" rpy="0.0 0.0 0.0" />
+        <dynamics damping="${joint_damping}"/>
+      </joint>
+    </xacro:unless>
     <link name="${arm_id}_link0">
       <visual>
@@ -28,9 +30,11 @@
         </geometry>
       </collision>
-      <inertial>
-        <origin xyz="0 0 0" rpy="0 0 0"/>
-        <mass value="3.06"/>
-        <inertia ixx="0.3" ixy="0.0" ixz="0.0" iyy="0.3" iyz="0.0" izz="0.3"/>
-      </inertial>
+      <xacro:unless value="${in_gazebo == 'false'}">
+        <inertial>
+          <origin xyz="0 0 0" rpy="0 0 0"/>
+          <mass value="3.06"/>
+          <inertia ixx="0.3" ixy="0.0" ixz="0.0" iyy="0.3" iyz="0.0" izz="0.3"/>
+        </inertial>
+      </xacro:unless>
     </link>
     <link name="${arm_id}_link1">
@@ -46,11 +50,11 @@
       </collision>
       <inertial>
-        <origin xyz="0 0 0" rpy="0 0 0"/>
-        <mass value="2.34"/>
-        <inertia ixx="0.3" ixy="0.0" ixz="0.0" iyy="0.3" iyz="0.0" izz="0.3"/>
+        <origin xyz="3.875e-03 2.081e-03 -0.1750" rpy="0 0 0"/>
+        <mass value="4.970684"/>
+        <inertia ixx="7.0337e-01" ixy="-1.3900e-04" ixz="6.7720e-03" iyy="7.0661e-01" iyz="1.9169e-02" izz="9.1170e-03"/>
       </inertial>
     </link>
     <joint name="${arm_id}_joint1" type="revolute">
-      <!-- <safety_controller k_position="100.0" k_velocity="40.0" soft_lower_limit="-2.8973" soft_upper_limit="2.8973"/> -->
+      <safety_controller k_position="100.0" k_velocity="40.0" soft_lower_limit="-2.8973" soft_upper_limit="2.8973"/>
       <origin rpy="0 0 0" xyz="0 0 0.333"/>
       <parent link="${arm_id}_link0"/>
@@ -72,11 +76,11 @@
       </collision>
       <inertial>
-        <origin xyz="0 0 0" rpy="0 0 0"/>
-        <mass value="2.36"/>
-        <inertia ixx="0.3" ixy="0.0" ixz="0.0" iyy="0.3" iyz="0.0" izz="0.3"/>
+        <origin xyz="-3.141e-03 -2.872e-02 3.495e-03" rpy="0 0 0"/>
+        <mass value="0.646926"/>
+        <inertia ixx="7.9620e-03" ixy="-3.9250e-03" ixz="1.0254e-02" iyy="2.8110e-02" iyz="7.0400e-04" izz="2.5995e-02"/>
       </inertial>
     </link>
     <joint name="${arm_id}_joint2" type="revolute">
-      <!-- <safety_controller k_position="100.0" k_velocity="40.0" soft_lower_limit="-1.7628" soft_upper_limit="1.7628"/> -->
+      <safety_controller k_position="100.0" k_velocity="40.0" soft_lower_limit="-1.7628" soft_upper_limit="1.7628"/>
       <origin rpy="${-pi/2} 0 0" xyz="0 0 0"/>
       <parent link="${arm_id}_link1"/>
@@ -98,11 +102,11 @@
       </collision>
       <inertial>
-        <origin xyz="0 0 0" rpy="0 0 0"/>
-        <mass value="2.38"/>
-        <inertia ixx="0.3" ixy="0.0" ixz="0.0" iyy="0.3" iyz="0.0" izz="0.3"/>
+        <origin xyz="2.7518e-02 3.9252e-02 -6.6502e-02" rpy="0 0 0"/>
+        <mass value="3.228604"/>
+        <inertia ixx="3.7242e-02" ixy="-4.7610e-03" ixz="-1.1396e-02" iyy="3.6155e-02" iyz="-1.2805e-02" izz="1.0830e-02"/>
       </inertial>
     </link>
     <joint name="${arm_id}_joint3" type="revolute">
-      <!-- <safety_controller k_position="100.0" k_velocity="40.0" soft_lower_limit="-2.8973" soft_upper_limit="2.8973"/> -->
+      <safety_controller k_position="100.0" k_velocity="40.0" soft_lower_limit="-2.8973" soft_upper_limit="2.8973"/>
       <origin rpy="${pi/2} 0 0" xyz="0 -0.316 0"/>
       <parent link="${arm_id}_link2"/>
@@ -124,11 +128,11 @@
       </collision>
       <inertial>
-        <origin xyz="0 0 0" rpy="0 0 0"/>
-        <mass value="2.43"/>
-        <inertia ixx="0.3" ixy="0.0" ixz="0.0" iyy="0.3" iyz="0.0" izz="0.3"/>
+        <origin xyz="-5.317e-02 1.04419e-01 2.7454e-02" rpy="0 0 0"/>
+        <mass value="3.587895"/>
+        <inertia ixx="2.5853e-02" ixy="7.7960e-03" ixz="-1.3320e-03" iyy="1.9552e-02" iyz="8.6410e-03" izz="2.8323e-02"/>
       </inertial>
     </link>
     <joint name="${arm_id}_joint4" type="revolute">
-      <!-- <safety_controller k_position="100.0" k_velocity="40.0" soft_lower_limit="-3.0718" soft_upper_limit="-0.0698"/> -->
+      <safety_controller k_position="100.0" k_velocity="40.0" soft_lower_limit="-3.0718" soft_upper_limit="-0.0698"/>
       <origin rpy="${pi/2} 0 0" xyz="0.0825 0 0"/>
       <parent link="${arm_id}_link3"/>
@@ -150,11 +154,11 @@
       </collision>
       <inertial>
-        <origin xyz="0 0 0" rpy="0 0 0"/>
-        <mass value="3.5"/>
-        <inertia ixx="0.3" ixy="0.0" ixz="0.0" iyy="0.3" iyz="0.0" izz="0.3"/>
+        <origin xyz="-1.1953e-02 4.1065e-02 -3.8437e-02" rpy="0 0 0"/>
+        <mass value="1.225946"/>
+        <inertia ixx="3.5549e-02" ixy="-2.1170e-03" ixz="-4.0370e-03" iyy="2.9474e-02" iyz="2.2900e-04" izz="8.6270e-03"/>
       </inertial>
     </link>
     <joint name="${arm_id}_joint5" type="revolute">
-      <!-- <safety_controller k_position="100.0" k_velocity="40.0" soft_lower_limit="-2.8973" soft_upper_limit="2.8973"/> -->
+      <safety_controller k_position="100.0" k_velocity="40.0" soft_lower_limit="-2.8973" soft_upper_limit="2.8973"/>
       <origin rpy="${-pi/2} 0 0" xyz="-0.0825 0.384 0"/>
       <parent link="${arm_id}_link4"/>
@@ -176,11 +180,11 @@
       </collision>
       <inertial>
-        <origin xyz="0 0 0" rpy="0 0 0"/>
-        <mass value="1.47"/>
-        <inertia ixx="0.3" ixy="0.0" ixz="0.0" iyy="0.3" iyz="0.0" izz="0.3"/>
+        <origin xyz="6.0149e-02 -1.4117e-02 -1.0517e-02" rpy="0 0 0"/>
+        <mass value="1.666555"/>
+        <inertia ixx="1.9640e-03" ixy="1.0900e-04" ixz="-1.1580e-03" iyy="4.3540e-03" iyz="3.4100e-04" izz="5.4330e-03"/>
       </inertial>
     </link>
     <joint name="${arm_id}_joint6" type="revolute">
-      <!-- <safety_controller k_position="100.0" k_velocity="40.0" soft_lower_limit="-0.0175" soft_upper_limit="3.7525"/> -->
+      <safety_controller k_position="100.0" k_velocity="40.0" soft_lower_limit="-0.0175" soft_upper_limit="3.7525"/>
       <origin rpy="${pi/2} 0 0" xyz="0 0 0"/>
       <parent link="${arm_id}_link5"/>
@@ -202,11 +206,11 @@
       </collision>
       <inertial>
-        <origin xyz="0 0 0" rpy="0 0 0"/>
-        <mass value="0.45"/>
-        <inertia ixx="0.3" ixy="0.0" ixz="0.0" iyy="0.3" iyz="0.0" izz="0.3"/>
+        <origin xyz="1.0517e-02 -4.252e-03 6.1597e-02" rpy="0 0 0"/>
+        <mass value="7.35522e-01"/>
+        <inertia ixx="1.2516e-02" ixy="-4.2800e-04" ixz="-1.1960e-03" iyy="1.0027e-02" iyz="-7.4100e-04" izz="4.8150e-03"/>
       </inertial>
     </link>
     <joint name="${arm_id}_joint7" type="revolute">
-      <!-- <safety_controller k_position="100.0" k_velocity="40.0" soft_lower_limit="-2.8973" soft_upper_limit="2.8973"/> -->
+      <safety_controller k_position="100.0" k_velocity="40.0" soft_lower_limit="-2.8973" soft_upper_limit="2.8973"/>
       <origin rpy="${pi/2} 0 0" xyz="0.088 0 0"/>
       <parent link="${arm_id}_link6"/>
@@ -220,5 +224,5 @@
         <origin xyz="0 0 0" rpy="0 0 0"/>
         <mass value="0.0"/>
-        <inertia ixx="0.3" ixy="0.0" ixz="0.0" iyy="0.3" iyz="0.0" izz="0.3"/>
+        <inertia ixx="0.001" ixy="0.0" ixz="0.0" iyy="0.001" iyz="0.0" izz="0.001"/>
       </inertial>
     </link>

File: robots/panda_arm_hand.urdf.xacro (robot description, xacro)
@@ -3,4 +3,5 @@
   <xacro:arg name="robot_name" default="panda"/>
   <xacro:arg name="load_gripper" default="true"/>
+  <xacro:arg name="load_gazebo" default="false"/>
   <xacro:include filename="$(find franka_panda_description)/robots/panda_arm.xacro"/>
   <xacro:if value="$(arg load_gripper)">
@@ -8,8 +9,13 @@
     <xacro:hand ns="panda" rpy="0 0 ${-pi/4}" connected_to="panda_link8"/>
   </xacro:if>
-  <xacro:include filename="$(find franka_panda_description)/robots/panda.gazebo.xacro"/>
-  <xacro:include filename="$(find franka_panda_description)/robots/panda.transmission.xacro"/>
-  <xacro:panda_arm />
-  <xacro:panda_gazebo robot_name="$(arg robot_name)" load_gripper="$(arg load_gripper)"/>
-  <xacro:panda_transmission robot_name="$(arg robot_name)" load_gripper="$(arg load_gripper)"/>
+  <xacro:if value="$(arg load_gazebo)">
+    <xacro:include filename="$(find franka_panda_description)/robots/panda.gazebo.xacro"/>
+    <xacro:include filename="$(find franka_panda_description)/robots/panda.transmission.xacro"/>
+    <xacro:panda_arm in_gazebo="true" />
+    <xacro:panda_gazebo robot_name="$(arg robot_name)" load_gripper="$(arg load_gripper)"/>
+    <xacro:panda_transmission robot_name="$(arg robot_name)" load_gripper="$(arg load_gripper)"/>
+  </xacro:if>
+  <xacro:unless value="$(arg load_gazebo)">
+    <xacro:panda_arm />
+  </xacro:unless>
 </robot>
