Commit message: add flag to use package with native gazebo ros control instead of panda_ros_control

File: robots/panda.transmission.xacro (robot description, xacro)
@@ -1,19 +1,25 @@
 <?xml version="1.0"?>
 <robot xmlns:xacro="http://www.ros.org/wiki/xacro">
-    <xacro:macro name="panda_transmission" params="robot_name load_gripper">
+    <xacro:macro name="panda_transmission" params="robot_name load_gripper use_gazebo_control">
         <!-- Load Gazebo lib and set the robot namespace -->
-        <gazebo>
-            <plugin name="panda_ros_control" filename="libpanda_gazebo_ros_control.so">
-                <robotNamespace></robotNamespace>
-                <robotSimType>panda_gazebo/PandaRobotHWSim</robotSimType>
-                <controlPeriod>0.001</controlPeriod>
-                <eStopTopic>sim_estop</eStopTopic>
-            </plugin>
-<!--             <plugin name="gazebo_ros_control" filename="libgazebo_ros_control.so">
-                <robotNamespace>/panda_simulator/</robotNamespace>
-                <robotSimType>gazebo_ros_control/DefaultRobotHWSim</robotSimType>
-                <legacyModeNS>true</legacyModeNS>
-              </plugin> -->
-        </gazebo>
+        <xacro:if value="${use_gazebo_control}">
+            <gazebo>
+                <plugin name="gazebo_ros_control" filename="libgazebo_ros_control.so">
+                    <robotNamespace>/</robotNamespace>
+                    <robotSimType>gazebo_ros_control/DefaultRobotHWSim</robotSimType>
+                    <legacyModeNS>true</legacyModeNS>
+                </plugin>
+            </gazebo>
+        </xacro:if>
+        <xacro:unless value="${use_gazebo_control}">
+            <gazebo>
+                <plugin name="panda_ros_control" filename="libpanda_gazebo_ros_control.so">
+                    <robotNamespace></robotNamespace>
+                    <robotSimType>panda_gazebo/PandaRobotHWSim</robotSimType>
+                    <controlPeriod>0.001</controlPeriod>
+                    <eStopTopic>sim_estop</eStopTopic>
+                </plugin>
+            </gazebo>
+        </xacro:unless>
         <transmission name="${robot_name}_tran_1">
             <type>transmission_interface/SimpleTransmission</type>

File: robots/panda_arm_hand.urdf.xacro (robot description, xacro)
@@ -4,4 +4,5 @@
   <xacro:arg name="load_gripper" default="true"/>
   <xacro:arg name="load_gazebo" default="false"/>
+  <xacro:arg name="use_gazebo_control" default="false"/>
   <xacro:include filename="$(find franka_panda_description)/robots/panda_arm.xacro"/>
   <xacro:if value="$(arg load_gripper)">
@@ -14,5 +15,5 @@
     <xacro:panda_arm in_gazebo="true" />
     <xacro:panda_gazebo robot_name="$(arg robot_name)" load_gripper="$(arg load_gripper)"/>
-    <xacro:panda_transmission robot_name="$(arg robot_name)" load_gripper="$(arg load_gripper)"/>
+    <xacro:panda_transmission robot_name="$(arg robot_name)" load_gripper="$(arg load_gripper)" use_gazebo_control="$(arg use_gazebo_control)"/>
   </xacro:if>
   <xacro:unless value="$(arg load_gazebo)">
