Commit message: using old collision mesh instead of the new ones; new franka_description collision seems to be buggy

File: robots/panda_arm.xacro (robot description, xacro)
@@ -1,5 +1,5 @@
 <?xml version='1.0'?>
 <robot xmlns:xacro="http://www.ros.org/wiki/xacro" name="panda">
-  <xacro:macro name="panda_arm" params="arm_id:='panda' description_pkg:='franka_description' connected_to:=''  in_gazebo='false' xyz:='0 0 0' rpy:='0 0 0'">
+  <xacro:macro name="panda_arm" params="arm_id:='panda' description_pkg:='franka_panda_description' connected_to:=''  in_gazebo='false' xyz:='0 0 0' rpy:='0 0 0'">
     <xacro:unless value="${not connected_to}">
       <joint name="${arm_id}_joint_${connected_to}" type="fixed">

Commit message: fixing #3;fix bug in connected_to param for using different parent frame for robot base

File: robots/panda_arm.xacro (robot description, xacro)
@@ -14,5 +14,10 @@
       <joint name="robot_to_world" type="fixed">
         <parent link="world" />
-        <child link="${arm_id}_link0" />
+        <xacro:if value="${not connected_to}">
+          <child link="${arm_id}_link0" />
+        </xacro:if>
+        <xacro:unless value="${not connected_to}">
+          <child link="${connected_to}"/>
+        </xacro:unless>
         <origin xyz="0.0 0.0 0.0" rpy="0.0 0.0 0.0" />
         <dynamics damping="${joint_damping}"/>

File: robots/panda_arm_hand.urdf.xacro (robot description, xacro)
@@ -5,4 +5,5 @@
   <xacro:arg name="load_gazebo" default="false"/>
   <xacro:arg name="use_gazebo_control" default="false"/>
+  <xacro:arg name="connected_to" default=""/>
   <xacro:include filename="$(find franka_panda_description)/robots/panda_arm.xacro"/>
   <xacro:if value="$(arg load_gripper)">
@@ -13,5 +14,5 @@
     <xacro:include filename="$(find franka_panda_description)/robots/panda.gazebo.xacro"/>
     <xacro:include filename="$(find franka_panda_description)/robots/panda.transmission.xacro"/>
-    <xacro:panda_arm in_gazebo="true" />
+    <xacro:panda_arm in_gazebo="true"  connected_to="$(arg connected_to)"/>
     <xacro:panda_gazebo robot_name="$(arg robot_name)" load_gripper="$(arg load_gripper)"/>
     <xacro:panda_transmission robot_name="$(arg robot_name)" load_gripper="$(arg load_gripper)" use_gazebo_control="$(arg use_gazebo_control)"/>

Commit message: removing 'world' link creation when using custom base frame

File: robots/panda_arm.xacro (robot description, xacro)
@@ -2,26 +2,20 @@
 <robot xmlns:xacro="http://www.ros.org/wiki/xacro" name="panda">
   <xacro:macro name="panda_arm" params="arm_id:='panda' description_pkg:='franka_panda_description' connected_to:=''  in_gazebo='false' xyz:='0 0 0' rpy:='0 0 0'">
-    <xacro:unless value="${not connected_to}">
-      <joint name="${arm_id}_joint_${connected_to}" type="fixed">
-        <parent link="${connected_to}"/>
-        <child link="${arm_id}_link0"/>
-        <origin rpy="${rpy}" xyz="${xyz}"/>
-      </joint>
+    <!-- If using custom frame with ${connected_to} param, make sure 'world' frame exists in its TF tree -->
+    <xacro:if value="${connected_to == ''}">
+      <link name="world" />
+      <xacro:property name="base_frame_name" value="world"/>
+    </xacro:if>
+    <xacro:unless value="${connected_to == ''}">
+      <xacro:property name="base_frame_name" value="${connected_to}"/>
     </xacro:unless>
-    <xacro:property name="joint_damping" value="1.0"/>
-    <xacro:unless value="${in_gazebo == 'false'}">
-      <link name="world" />
-      <joint name="robot_to_world" type="fixed">
-        <parent link="world" />
-        <xacro:if value="${not connected_to}">
-          <child link="${arm_id}_link0" />
-        </xacro:if>
-        <xacro:unless value="${not connected_to}">
-          <child link="${connected_to}"/>
-        </xacro:unless>
-        <origin xyz="0.0 0.0 0.0" rpy="0.0 0.0 0.0" />
-        <dynamics damping="${joint_damping}"/>
-      </joint>
-    </xacro:unless>
+    <joint name="${arm_id}_to_${base_frame_name}" type="fixed">
+      <parent link="${base_frame_name}"/>
+      <child link="${arm_id}_link0"/>
+      <origin rpy="${rpy}" xyz="${xyz}"/>
+      <xacro:unless value="${in_gazebo == 'false'}">
+        <dynamics damping="1.0"/>
+      </xacro:unless>
+    </joint>
     <link name="${arm_id}_link0">
       <visual>

File: robots/panda_arm_hand.urdf.xacro (robot description, xacro)
@@ -5,5 +5,5 @@
   <xacro:arg name="load_gazebo" default="false"/>
   <xacro:arg name="use_gazebo_control" default="false"/>
-  <xacro:arg name="connected_to" default=""/>
+  <xacro:arg name="connected_to" default=""/> <!-- If using a different frame with ${connected_to} param, make sure 'world' frame exists in the TF tree -->
   <xacro:include filename="$(find franka_panda_description)/robots/panda_arm.xacro"/>
   <xacro:if value="$(arg load_gripper)">

Commit message: reverting to old dynamics values for robot joints to fix joint velocity and torque issue (see issue #5)

File: robots/panda_arm.xacro (robot description, xacro)
@@ -227,5 +227,5 @@
     </link>
     <joint name="${arm_id}_joint8" type="fixed">
-      <origin rpy="0 0 0" xyz="0 0 0.107"/>
+    <origin rpy="0 0 0" xyz="0 0 0.107"/>
       <parent link="${arm_id}_link7"/>
       <child link="${arm_id}_link8"/>

Commit message: reverting dynamics values to fix #5

File: robots/panda_arm.xacro (robot description, xacro)
@@ -31,7 +31,7 @@
       <xacro:unless value="${in_gazebo == 'false'}">
         <inertial>
-          <origin rpy="0 0 0" xyz="-0.025566 -2.88e-05 0.057332"/>
-          <mass value="2.92"/>
-          <inertia ixx="0.00782229414331" ixy="-1.56191622996e-05" ixz="-0.00126005738123" iyy="0.0109027971813" iyz="1.08233858202e-05" izz="0.0102355503949"/>
+          <origin xyz="0 0 0" rpy="0 0 0"/>
+          <mass value="3.06"/>
+          <inertia ixx="0.3" ixy="0.0" ixz="0.0" iyy="0.3" iyz="0.0" izz="0.3"/>
         </inertial>
       </xacro:unless>
@@ -49,7 +49,7 @@
       </collision>
       <inertial>
-        <origin rpy="0 0 0" xyz="0 -0.0324958 -0.0675818"/>
-        <mass value="2.74"/>
-        <inertia ixx="0.0180416958283" ixy="0" ixz="0" iyy="0.0159136071891" iyz="0.0046758424612" izz="0.00620690827127"/>
+        <origin xyz="3.875e-03 2.081e-03 -0.1750" rpy="0 0 0"/>
+        <mass value="4.970684"/>
+        <inertia ixx="7.0337e-01" ixy="-1.3900e-04" ixz="6.7720e-03" iyy="7.0661e-01" iyz="1.9169e-02" izz="9.1170e-03"/>
       </inertial>
     </link>
@@ -75,7 +75,7 @@
       </collision>
       <inertial>
-        <origin rpy="0 0 0" xyz="0 -0.06861 0.0322285"/>
-        <mass value="2.74"/>
-        <inertia ixx="0.0182856182281" ixy="0" ixz="0" iyy="0.00621358421175" iyz="-0.00472844221905" izz="0.0161514346309"/>
+        <origin xyz="-3.141e-03 -2.872e-02 3.495e-03" rpy="0 0 0"/>
+        <mass value="0.646926"/>
+        <inertia ixx="7.9620e-03" ixy="-3.9250e-03" ixz="1.0254e-02" iyy="2.8110e-02" iyz="7.0400e-04" izz="2.5995e-02"/>
       </inertial>
     </link>
@@ -101,7 +101,7 @@
       </collision>
       <inertial>
-        <origin rpy="0 0 0" xyz="0.0469893 0.0316374 -0.031704"/>
-        <mass value="2.38"/>
-        <inertia ixx="0.00771376630908" ixy="-0.00248490625138" ixz="-0.00332147581033" iyy="0.00989108008727" iyz="-0.00217796151484" izz="0.00811723558464"/>
+        <origin xyz="2.7518e-02 3.9252e-02 -6.6502e-02" rpy="0 0 0"/>
+        <mass value="3.228604"/>
+        <inertia ixx="3.7242e-02" ixy="-4.7610e-03" ixz="-1.1396e-02" iyy="3.6155e-02" iyz="-1.2805e-02" izz="1.0830e-02"/>
       </inertial>
     </link>
@@ -127,7 +127,7 @@
       </collision>
       <inertial>
-        <origin rpy="0 0 0" xyz="-0.0360446 0.0336853 0.031882"/>
-        <mass value="2.38"/>
-        <inertia ixx="0.00799663881132" ixy="0.00347095570217" ixz="-0.00241222942995" iyy="0.00825390705278" iyz="0.00235774044121" izz="0.0102515004345"/>
+        <origin xyz="-5.317e-02 1.04419e-01 2.7454e-02" rpy="0 0 0"/>
+        <mass value="3.587895"/>
+        <inertia ixx="2.5853e-02" ixy="7.7960e-03" ixz="-1.3320e-03" iyy="1.9552e-02" iyz="8.6410e-03" izz="2.8323e-02"/>
       </inertial>
     </link>
@@ -153,7 +153,7 @@
       </collision>
       <inertial>
-        <origin rpy="0 0 0" xyz="0 0.0610427 -0.104176"/>
-        <mass value="2.74"/>
-        <inertia ixx="0.030371374513" ixy="6.50283587108e-07" ixz="-1.05129179916e-05" iyy="0.0288752887402" iyz="-0.00775653445787" izz="0.00444134056164"/>
+        <origin xyz="-1.1953e-02 4.1065e-02 -3.8437e-02" rpy="0 0 0"/>
+        <mass value="1.225946"/>
+        <inertia ixx="3.5549e-02" ixy="-2.1170e-03" ixz="-4.0370e-03" iyy="2.9474e-02" iyz="2.2900e-04" izz="8.6270e-03"/>
       </inertial>
     </link>
@@ -179,7 +179,7 @@
       </collision>
       <inertial>
-        <origin rpy="0 0 0" xyz="0.0510509 0.009108 0.0106343"/>
-        <mass value="1.55"/>
-        <inertia ixx="0.00303336450376" ixy="-0.000437276865508" ixz="0.000629257294877" iyy="0.00404479911567" iyz="0.000130472021025" izz="0.00558234286039"/>
+        <origin xyz="6.0149e-02 -1.4117e-02 -1.0517e-02" rpy="0 0 0"/>
+        <mass value="1.666555"/>
+        <inertia ixx="1.9640e-03" ixy="1.0900e-04" ixz="-1.1580e-03" iyy="4.3540e-03" iyz="3.4100e-04" izz="5.4330e-03"/>
       </inertial>
     </link>
@@ -205,7 +205,7 @@
       </collision>
       <inertial>
-        <origin rpy="0 0 0" xyz="0.0109695 0.0107965 0.0650411"/>
-        <mass value="0.54"/>
-        <inertia ixx="0.000888868887021" ixy="-0.00012239074652" ixz="3.98699829666e-05" iyy="0.000888001373233" iyz="-9.33825115206e-05" izz="0.0007176834609"/>
+        <origin xyz="1.0517e-02 -4.252e-03 6.1597e-02" rpy="0 0 0"/>
+        <mass value="7.35522e-01"/>
+        <inertia ixx="1.2516e-02" ixy="-4.2800e-04" ixz="-1.1960e-03" iyy="1.0027e-02" iyz="-7.4100e-04" izz="4.8150e-03"/>
       </inertial>
     </link>
@@ -221,7 +221,7 @@
     <link name="${arm_id}_link8">
       <inertial>
-        <origin rpy="0 0 0" xyz="0 0 0"/>
+        <origin xyz="0 0 0" rpy="0 0 0"/>
         <mass value="0.0"/>
-        <inertia ixx="0.0" ixy="0.0" ixz="0.0" iyy="0.0" iyz="0.0" izz="0.0"/>
+        <inertia ixx="0.001" ixy="0.0" ixz="0.0" iyy="0.001" iyz="0.0" izz="0.001"/>
       </inertial>
     </link>
