Commit message: Split collision geometry into three separate meshes for link5

File: robots/panda_arm.urdf (robot description, URDF)
Before this commit: robot panda, 9 links, 8 joints
Links:
- link panda_link5: geometry collision mesh filename=package://${description_pkg}/meshes/collision/link5_1.stl; collision mesh filename=package://${description_pkg}/meshes/collision/link5_2.stl

File: robots/panda_arm.xacro (robot description, xacro)
@@ -149,5 +149,15 @@
       <collision>
         <geometry>
-          <mesh filename="package://${description_pkg}/meshes/collision/link5.stl"/>
+          <mesh filename="package://${description_pkg}/meshes/collision/link5_1.stl"/>
+        </geometry>
+      </collision>
+      <collision>
+        <geometry>
+          <mesh filename="package://${description_pkg}/meshes/collision/link5_2.stl"/>
+        </geometry>
+      </collision>
+      <collision>
+        <geometry>
+          <mesh filename="package://${description_pkg}/meshes/collision/link5_3.stl"/>
         </geometry>
       </collision>
